File: KiCAD/eegw:ads1299/eegw:ads1299.kicad_sch (KiCad schematic)
At the start: 35 parts, among them J1 ESP32-L, J10 ESP32-R2, J2 ESP32-L3, J3 ESP32-L2, J4 ESP32_Left, J5 ESP32_Right, J6 ESP32-R, J9 gpioADS, U1 ADS1299IPAG

Commit message: updated kicad renumbered
Parts:
- renumbered C24 to C1, C5 to C12, C22 to C13, C19 to C16, C20 to C17, C10 to C19, C3 to C2, C17 to C20, C23 to C28, C6 to C3, C21 to C9, J4 to J3, J6 to J4, J3 to J6, J10 to J7, J9 to J8, JP4 to JP1, JP3 to JP2, JP2 to JP3, JP1 to JP4, R30 to R11, R29 to R14, R26 to R15, R25 to R16, R79 to R17, R80 to R18, R82 to R19, R28 to R20, R81 to R21, R27 to R22
Changed lines of the file:
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@@
 		(on_board yes)
 		(dnp no)
-		(property "Reference" "C19"
+		(property "Reference" "C16"
 			(at 29.718 128.524 0)
 			(effects
@@
 			(project "eegw:ads1299"
 				(path "/3f21101e-7933-421f-83b1-297c54584233"
-					(reference "C19")
+					(reference "C16")
 					(unit 1)
 				)
@@
 		(dnp no)
 		(fields_autoplaced yes)
-		(property "Reference" "J9"
+		(property "Reference" "J8"
 			(at 240.03 20.3199 0)
 			(effects
@@
 			(project ""
 				(path "/3f21101e-7933-421f-83b1-297c54584233"
-					(reference "J9")
+					(reference "J8")
 					(unit 1)
 				)
@@
 		(on_board yes)
 		(dnp no)
-		(property "Reference" "J4"
+		(property "Reference" "J3"
 			(at 224.028 110.236 0)
 			(effects
@@
 			(project "eegw:ads1299"
 				(path "/3f21101e-7933-421f-83b1-297c54584233"
-					(reference "J4")
+					(reference "J3")
 					(unit 1)
 				)
@@
 		(on_board yes)
 		(dnp no)
-		(property "Reference" "C21"
+		(property "Reference" "C9"
 			(at 54.356 125.73 90)
 			(effects
@@
 			(project "eegw:ads1299"
 				(path "/3f21101e-7933-421f-83b1-297c54584233"
-					(reference "C21")
+					(reference "C9")
 					(unit 1)
 				)
@@
 		(on_board yes)
 		(dnp no)
-		(property "Reference" "JP4"
+		(property "Reference" "JP1"
 			(at 183.896 56.642 0)
 			(effects
@@
 			(project "eegw:ads1299"
 				(path "/3f21101e-7933-421f-83b1-297c54584233"
-					(reference "JP4")
+					(reference "JP1")
 					(unit 1)
 				)
@@
 		(dnp no)
 		(fields_autoplaced yes)
-		(property "Reference" "R26"
+		(property "Reference" "R15"
 			(at 256.54 31.7499 0)
 			(effects
@@
 			(project "eegw:ads1299"
 				(path "/3f21101e-7933-421f-83b1-297c54584233"
-					(reference "R26")
+					(reference "R15")
 					(unit 1)
 				)
@@
 		(on_board yes)
 		(dnp no)
-		(property "Reference" "C10"
+		(property "Reference" "C19"
 			(at 104.902 36.068 0)
 			(effects
@@
 			(project "eegw:ads1299"
 				(path "/3f21101e-7933-421f-83b1-297c54584233"
-					(reference "C10")
+					(reference "C19")
 					(unit 1)
 				)
@@
 		(on_board yes)
 		(dnp no)
-		(property "Reference" "C23"
+		(property "Reference" "C28"
 			(at 67.564 133.858 0)
 			(effects
@@
 			(project "eegw:ads1299"
 				(path "/3f21101e-7933-421f-83b1-297c54584233"
-					(reference "C23")
+					(reference "C28")
 					(unit 1)
 				)
@@
 		(on_board yes)
 		(dnp no)
-		(property "Reference" "R80"
+		(property "Reference" "R18"
 			(at 198.12 32.004 90)
 			(effects
@@
 			(project "eegw:ads1299"
 				(path "/3f21101e-7933-421f-83b1-297c54584233"
-					(reference "R80")
+					(reference "R18")
 					(unit 1)
 				)
@@
 		(on_board yes)
 		(dnp no)
-		(property "Reference" "C5"
+		(property "Reference" "C12"
 			(at 68.072 38.608 0)
 			(effects
@@
 			(project "eegw:ads1299"
 				(path "/3f21101e-7933-421f-83b1-297c54584233"
-					(reference "C5")
+					(reference "C12")
 					(unit 1)
 				)
@@
 		(on_board yes)
 		(dnp no)
-		(property "Reference" "C3"
+		(property "Reference" "C2"
 			(at 59.182 38.608 0)
 			(effects
@@
 			(project "eegw:ads1299"
 				(path "/3f21101e-7933-421f-83b1-297c54584233"
-					(reference "C3")
+					(reference "C2")
 					(unit 1)
 				)
@@
 		(on_board yes)
 		(dnp no)
-		(property "Reference" "C24"
+		(property "Reference" "C1"
 			(at 151.638 57.15 0)
 			(effects
@@
 			(project ""
 				(path "/3f21101e-7933-421f-83b1-297c54584233"
-					(reference "C24")
+					(reference "C1")
 					(unit 1)
 				)
@@
 		(on_board yes)
 		(dnp no)
-		(property "Reference" "JP3"
+		(property "Reference" "JP2"
 			(at 184.15 44.45 0)
 			(effects
@@
 			(project "eegw:ads1299"
 				(path "/3f21101e-7933-421f-83b1-297c54584233"
-					(reference "JP3")
+					(reference "JP2")
 					(unit 1)
 				)
@@
 		(on_board yes)
 		(dnp no)
-		(property "Reference" "C20"
+		(property "Reference" "C17"
 			(at 42.418 128.524 0)
 			(effects
@@
 			(project "eegw:ads1299"
 				(path "/3f21101e-7933-421f-83b1-297c54584233"
-					(reference "C20")
+					(reference "C17")
 					(unit 1)
 				)
@@
 		(on_board yes)
 		(dnp no)
-		(property "Reference" "R30"
+		(property "Reference" "R11"
 			(at 139.954 57.15 0)
 			(effects
@@
 			(project ""
 				(path "/3f21101e-7933-421f-83b1-297c54584233"
-					(reference "R30")
+					(reference "R11")
 					(unit 1)
 				)
@@
 		(on_board yes)
 		(dnp no)
-		(property "Reference" "C6"
+		(property "Reference" "C3"
 			(at 113.792 36.068 0)
 			(effects
@@
 			(project "eegw:ads1299"
 				(path "/3f21101e-7933-421f-83b1-297c54584233"
-					(reference "C6")
+					(reference "C3")
 					(unit 1)
 				)
@@
 		(on_board yes)
 		(dnp no)
-		(property "Reference" "R82"
+		(property "Reference" "R19"
 			(at 198.12 57.404 90)
 			(effects
@@
 			(project "eegw:ads1299"
 				(path "/3f21101e-7933-421f-83b1-297c54584233"
-					(reference "R82")
+					(reference "R19")
 					(unit 1)
 				)
@@
 		(dnp no)
 		(fields_autoplaced yes)
-		(property "Reference" "R27"
+		(property "Reference" "R22"
 			(at 273.05 21.5899 0)
 			(effects
@@
 			(project "eegw:ads1299"
 				(path "/3f21101e-7933-421f-83b1-297c54584233"
-					(reference "R27")
+					(reference "R22")
 					(unit 1)
 				)
@@
 		(on_board yes)
 		(dnp no)
-		(property "Reference" "R29"
+		(property "Reference" "R14"
 			(at 144.78 110.4899 0)
 			(effects
@@
 			(project ""
 				(path "/3f21101e-7933-421f-83b1-297c54584233"
-					(reference "R29")
+					(reference "R14")
 					(unit 1)
 				)
@@
 		(on_board yes)
 		(dnp no)
-		(property "Reference" "JP2"
+		(property "Reference" "JP3"
 			(at 184.15 31.496 0)
 			(effects
@@
 			(project "eegw:ads1299"
 				(path "/3f21101e-7933-421f-83b1-297c54584233"
-					(reference "JP2")
+					(reference "JP3")
 					(unit 1)
 				)
@@
 		(dnp no)
 		(fields_autoplaced yes)
-		(property "Reference" "R28"
+		(property "Reference" "R20"
 			(at 273.05 31.7499 0)
 			(effects
@@
 			(project "eegw:ads1299"
 				(path "/3f21101e-7933-421f-83b1-297c54584233"
-					(reference "R28")
+					(reference "R20")
 					(unit 1)
 				)
@@
 		(dnp no)
 		(fields_autoplaced yes)
-		(property "Reference" "R25"
+		(property "Reference" "R16"
 			(at 256.54 21.5899 0)
 			(effects
@@
 			(project ""
 				(path "/3f21101e-7933-421f-83b1-297c54584233"
-					(reference "R25")
+					(reference "R16")
 					(unit 1)
 				)
@@
 		(on_board yes)
 		(dnp no)
-		(property "Reference" "R81"
+		(property "Reference" "R21"
 			(at 198.12 44.704 90)
 			(effects
@@
 			(project "eegw:ads1299"
 				(path "/3f21101e-7933-421f-83b1-297c54584233"
-					(reference "R81")
+					(reference "R21")
 					(unit 1)
 				)
@@
 		(on_board yes)
 		(dnp no)
-		(property "Reference" "J3"
+		(property "Reference" "J6"
 			(at 193.04 136.398 0)
 			(effects
@@
 			(project "eegw:ads1299"
 				(path "/3f21101e-7933-421f-83b1-297c54584233"
-					(reference "J3")
+					(reference "J6")
 					(unit 1)
 				)
@@
 		(on_board yes)
 		(dnp no)
-		(property "Reference" "J6"
+		(property "Reference" "J4"
 			(at 275.844 111.76 0)
 			(effects
@@
 			(project "eegw:ads1299"
 				(path "/3f21101e-7933-421f-83b1-297c54584233"
-					(reference "J6")
+					(reference "J4")
 					(unit 1)
 				)
@@
 		(on_board yes)
 		(dnp no)
-		(property "Reference" "C17"
+		(property "Reference" "C20"
 			(at 50.292 113.03 90)
 			(effects
@@
 			(project ""
 				(path "/3f21101e-7933-421f-83b1-297c54584233"
-					(reference "C17")
+					(reference "C20")
 					(unit 1)
 				)
@@
 		(on_board yes)
 		(dnp no)
-		(property "Reference" "J10"
+		(property "Reference" "J7"
 			(at 274.574 131.572 0)
 			(effects
@@
 			(project ""
 				(path "/3f21101e-7933-421f-83b1-297c54584233"
-					(reference "J10")
+					(reference "J7")
 					(unit 1)
 				)
@@
 		(on_board yes)
 		(dnp no)
-		(property "Reference" "C22"
+		(property "Reference" "C13"
 			(at 60.198 133.604 0)
 			(effects
@@
 			(project "eegw:ads1299"
 				(path "/3f21101e-7933-421f-83b1-297c54584233"
-					(reference "C22")
+					(reference "C13")
 					(unit 1)
 				)
@@
 		(on_board yes)
 		(dnp no)
-		(property "Reference" "JP1"
+		(property "Reference" "JP4"
 			(at 184.404 18.796 0)
 			(effects
@@
 			(project ""
 				(path "/3f21101e-7933-421f-83b1-297c54584233"
-					(reference "JP1")
+					(reference "JP4")
 					(unit 1)
 				)
@@
 		(on_board yes)
 		(dnp no)
-		(property "Reference" "R79"
+		(property "Reference" "R17"
 			(at 198.12 19.304 90)
 			(effects
@@
 			(project ""
 				(path "/3f21101e-7933-421f-83b1-297c54584233"
-					(reference "R79")
+					(reference "R17")
 					(unit 1)
 				)
