File: Hardware/KiCAD/new_kicad/eegw:ads1299/tpd4e1b06.kicad_sch (KiCad schematic)
At the start: 18 parts, among them J4 L, J6 R

Commit message: update filled zone & geograpgically annotated pcb
Parts:
- C1: renamed from C4; footprint CKCL44_TDK -> Capacitor_SMD:CKCL44_TDK
- C17: renamed from C10; footprint CKCL44_TDK -> Capacitor_SMD:CKCL44_TDK
- C5: footprint CKCL44_TDK -> Capacitor_SMD:CKCL44_TDK
- C6: renamed from C7; footprint CKCL44_TDK -> Capacitor_SMD:CKCL44_TDK
- C7: renamed from C6; footprint CKCL44_TDK -> Capacitor_SMD:CKCL44_TDK
- J7: renamed from J4; value L -> N
- J8: renamed from J6; value R -> P
- renumbered R7 to R1, R13 to R10, R9 to R5, R10 to R6, R8 to R7, U2 to U1, U4 to U2, U6 to U3, U5 to U4, U3 to U5, U8 to U7
Changed lines of the file:
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@@
 		(dnp no)
 		(fields_autoplaced yes)
-		(property "Reference" "C4"
+		(property "Reference" "C1"
 			(at 105.41 40.6399 0)
 			(effects
@@
 			)
 		)
-		(property "Footprint" "CKCL44_TDK"
+		(property "Footprint" "Capacitor_SMD:CKCL44_TDK"
 			(at 86.36 38.1 0)
 			(effects
@@
 			(project ""
 				(path "/3f21101e-7933-421f-83b1-297c54584233/f02e0be0-6bc7-41d9-a052-1a2d3a081560"
-					(reference "C4")
+					(reference "C1")
 					(unit 1)
 				)
@@
 		(dnp no)
 		(fields_autoplaced yes)
-		(property "Reference" "R8"
+		(property "Reference" "R7"
 			(at 76.2 64.77 0)
 			(effects
@@
 			(project "eegw:ads1299"
 				(path "/3f21101e-7933-421f-83b1-297c54584233/f02e0be0-6bc7-41d9-a052-1a2d3a081560"
-					(reference "R8")
+					(reference "R7")
 					(unit 1)
 				)
@@
 		(on_board yes)
 		(dnp no)
-		(property "Reference" "U4"
+		(property "Reference" "U2"
 			(at 147.066 96.012 0)
 			(effects
@@
 			(project "eegw:ads1299"
 				(path "/3f21101e-7933-421f-83b1-297c54584233/f02e0be0-6bc7-41d9-a052-1a2d3a081560"
-					(reference "U4")
+					(reference "U2")
 					(unit 1)
 				)
@@
 		(dnp no)
 		(fields_autoplaced yes)
-		(property "Reference" "R10"
+		(property "Reference" "R6"
 			(at 77.47 156.21 0)
 			(effects
@@
 			(project "eegw:ads1299"
 				(path "/3f21101e-7933-421f-83b1-297c54584233/f02e0be0-6bc7-41d9-a052-1a2d3a081560"
-					(reference "R10")
+					(reference "R6")
 					(unit 1)
 				)
@@
 		(on_board yes)
 		(dnp no)
-		(property "Reference" "J4"
+		(property "Reference" "J7"
 			(at 235.458 96.012 0)
 			(effects
@@
 			)
 		)
-		(property "Value" "L"
+		(property "Value" "N"
 			(at 236.474 99.06 0)
 			(effects
@@
 			(project "eegw:ads1299"
 				(path "/3f21101e-7933-421f-83b1-297c54584233/f02e0be0-6bc7-41d9-a052-1a2d3a081560"
-					(reference "J4")
+					(reference "J7")
 					(unit 1)
 				)
@@
 		(dnp no)
 		(fields_autoplaced yes)
-		(property "Reference" "R9"
+		(property "Reference" "R5"
 			(at 76.2 110.49 0)
 			(effects
@@
 			(project "eegw:ads1299"
 				(path "/3f21101e-7933-421f-83b1-297c54584233/f02e0be0-6bc7-41d9-a052-1a2d3a081560"
-					(reference "R9")
+					(reference "R5")
 					(unit 1)
 				)
@@
 		(on_board yes)
 		(dnp no)
-		(property "Reference" "U2"
+		(property "Reference" "U1"
 			(at 41.656 22.352 0)
 			(effects
@@
 			(project ""
 				(path "/3f21101e-7933-421f-83b1-297c54584233/f02e0be0-6bc7-41d9-a052-1a2d3a081560"
-					(reference "U2")
+					(reference "U1")
 					(unit 1)
 				)
@@
 		(on_board yes)
 		(dnp no)
-		(property "Reference" "U6"
+		(property "Reference" "U3"
 			(at 42.926 160.782 0)
 			(effects
@@
 			(project "eegw:ads1299"
 				(path "/3f21101e-7933-421f-83b1-297c54584233/f02e0be0-6bc7-41d9-a052-1a2d3a081560"
-					(reference "U6")
+					(reference "U3")
 					(unit 1)
 				)
@@
 		(dnp no)
 		(fields_autoplaced yes)
-		(property "Reference" "C10"
+		(property "Reference" "C17"
 			(at 246.38 49.5299 0)
 			(effects
@@
 			)
 		)
-		(property "Footprint" "CKCL44_TDK"
+		(property "Footprint" "Capacitor_SMD:CKCL44_TDK"
 			(at 227.33 46.99 0)
 			(effects
@@
 			(project "eegw:ads1299"
 				(path "/3f21101e-7933-421f-83b1-297c54584233/f02e0be0-6bc7-41d9-a052-1a2d3a081560"
-					(reference "C10")
+					(reference "C17")
 					(unit 1)
 				)
@@
 		(on_board yes)
 		(dnp no)
-		(property "Reference" "J6"
+		(property "Reference" "J8"
 			(at 255.524 96.52 0)
 			(effects
@@
 			)
 		)
-		(property "Value" "R"
+		(property "Value" "P"
 			(at 256.286 99.314 0)
 			(effects
@@
 			(project "eegw:ads1299"
 				(path "/3f21101e-7933-421f-83b1-297c54584233/f02e0be0-6bc7-41d9-a052-1a2d3a081560"
-					(reference "J6")
+					(reference "J8")
 					(unit 1)
 				)
@@
 			)
 		)
-		(property "Footprint" "CKCL44_TDK"
+		(property "Footprint" "Capacitor_SMD:CKCL44_TDK"
 			(at 86.36 85.09 0)
 			(effects
@@
 		(dnp no)
 		(fields_autoplaced yes)
-		(property "Reference" "C7"
+		(property "Reference" "C6"
 			(at 106.68 179.0699 0)
 			(effects
@@
 			)
 		)
-		(property "Footprint" "CKCL44_TDK"
+		(property "Footprint" "Capacitor_SMD:CKCL44_TDK"
 			(at 87.63 176.53 0)
 			(effects
@@
 			(project "eegw:ads1299"
 				(path "/3f21101e-7933-421f-83b1-297c54584233/f02e0be0-6bc7-41d9-a052-1a2d3a081560"
-					(reference "C7")
+					(reference "C6")
 					(unit 1)
 				)
@@
 		(dnp no)
 		(fields_autoplaced yes)
-		(property "Reference" "R7"
+		(property "Reference" "R1"
 			(at 76.2 17.78 0)
 			(effects
@@
 			(project ""
 				(path "/3f21101e-7933-421f-83b1-297c54584233/f02e0be0-6bc7-41d9-a052-1a2d3a081560"
-					(reference "R7")
+					(reference "R1")
 					(unit 1)
 				)
@@
 		(on_board yes)
 		(dnp no)
-		(property "Reference" "U3"
+		(property "Reference" "U5"
 			(at 41.656 69.342 0)
 			(effects
@@
 			(project "eegw:ads1299"
 				(path "/3f21101e-7933-421f-83b1-297c54584233/f02e0be0-6bc7-41d9-a052-1a2d3a081560"
-					(reference "U3")
+					(reference "U5")
 					(unit 1)
 				)
@@
 		(on_board yes)
 		(dnp no)
-		(property "Reference" "U8"
+		(property "Reference" "U7"
 			(at 182.626 31.242 0)
 			(effects
@@
 			(project "eegw:ads1299"
 				(path "/3f21101e-7933-421f-83b1-297c54584233/f02e0be0-6bc7-41d9-a052-1a2d3a081560"
-					(reference "U8")
+					(reference "U7")
 					(unit 1)
 				)
@@
 		(on_board yes)
 		(dnp no)
-		(property "Reference" "U5"
+		(property "Reference" "U4"
 			(at 41.656 115.062 0)
 			(effects
@@
 			(project "eegw:ads1299"
 				(path "/3f21101e-7933-421f-83b1-297c54584233/f02e0be0-6bc7-41d9-a052-1a2d3a081560"
-					(reference "U5")
+					(reference "U4")
 					(unit 1)
 				)
@@
 		(dnp no)
 		(fields_autoplaced yes)
-		(property "Reference" "C6"
+		(property "Reference" "C7"
 			(at 105.41 133.3499 0)
 			(effects
@@
 			)
 		)
-		(property "Footprint" "CKCL44_TDK"
+		(property "Footprint" "Capacitor_SMD:CKCL44_TDK"
 			(at 86.36 130.81 0)
 			(effects
@@
 			(project "eegw:ads1299"
 				(path "/3f21101e-7933-421f-83b1-297c54584233/f02e0be0-6bc7-41d9-a052-1a2d3a081560"
-					(reference "C6")
+					(reference "C7")
 					(unit 1)
 				)
@@
 		(dnp no)
 		(fields_autoplaced yes)
-		(property "Reference" "R13"
+		(property "Reference" "R10"
 			(at 217.17 26.67 0)
 			(effects
@@
 			(project "eegw:ads1299"
 				(path "/3f21101e-7933-421f-83b1-297c54584233/f02e0be0-6bc7-41d9-a052-1a2d3a081560"
-					(reference "R13")
-					(unit 1)
-				)
+					(reference "R10")
+					(unit 1)
+				)
